Commit message: Refactoring m2020 URDF for Development

File: rover/m2020.urdf (robot description, URDF)
Before this commit: robot Perseverance, 115 links, 114 joints
Links:
- link Body_BogieLeft: mass 0 -> 12.0000
- link Body_BogieRight: mass 0 -> 12.0000
- link Body_Chassis: mass 0 -> 670.0000
- link Body_CorerFeed: mass 0 -> 30.0000
- link Body_Differential: mass 0 -> 8.0000
- link Body_HGA_AZ: mass 0 -> 1.0000
- link Body_HGA_EL: mass 0 -> 4.0000
- link Body_MHS_DebrisShield: mass 0 -> 2.0000
- link Body_RA_Base: mass 0 -> 4.0000
- link Body_RA_Link1: mass 0 -> 7.0000
- link Body_RA_Link2: mass 0 -> 6.0000
- link Body_RA_Link3: mass 0 -> 5.0000
- link Body_RA_Link4: mass 0 -> 4.0000
- link Body_RA_Link5: mass 0 -> 3.0000
- link Body_RSM_AZ: mass 0 -> 2.0000
- link Body_RSM_EL: mass 0 -> 8.0000
- link Body_RockerLeft: mass 0 -> 18.0000
- link Body_RockerRight: mass 0 -> 18.0000
- link Body_SHERLOC_Cap: mass 0 -> 3.0000
- link Body_StabilizerFar: mass 0 -> 2.0000
- link Body_StabilizerNear: mass 0 -> 2.0000
- link Body_SteerLeftFront: mass 0 -> 4.0000
- link Body_SteerLeftRear: mass 0 -> 4.0000
- link Body_SteerRightFront: mass 0 -> 4.0000
- link Body_SteerRightRear: mass 0 -> 4.0000
- link Body_Turret: mass 0 -> 5.0000
- link Body_WATSON_Cap: mass 0 -> 3.0000
- link Body_WheelLeftFront: mass 0 -> 30.0000
- link Body_WheelLeftMiddle: mass 0 -> 30.0000
- link Body_WheelLeftRear: mass 0 -> 30.0000
- link Body_WheelRightFront: mass 0 -> 30.0000
- link Body_WheelRightMiddle: mass 0 -> 30.0000
- link Body_WheelRightRear: mass 0 -> 30.0000
- link Frame_ANT: mass 0 -> 0.0100
- link Frame_ATS1: mass 0 -> 0.0100
- link Frame_ATS2: mass 0 -> 0.0100
- link Frame_ATS3: mass 0 -> 0.0100
- link Frame_ATS4: mass 0 -> 0.0100
- link Frame_ATS5: mass 0 -> 0.0100
- link Frame_BOGIE_L: mass 0 -> 0.0100
- link Frame_BOGIE_R: mass 0 -> 0.0100
- link Frame_CAL_MC1: mass 0 -> 0.0100
- link Frame_CAL_MC2: mass 0 -> 0.0100
- link Frame_CAL_PIXL: mass 0 -> 0.0100
- link Frame_CAL_SC: mass 0 -> 0.0100
- link Frame_CAL_SHERLOC: mass 0 -> 0.0100
- link Frame_DIFF: mass 0 -> 0.0100
- link Frame_DOCKING_POST: mass 0 -> 0.0100
- link Frame_DRILL: mass 0 -> 0.0100
- link Frame_FCS: mass 0 -> 0.0100
- link Frame_FHC1: mass 0 -> 0.0100
- link Frame_FHC1_FOV: mass 0 -> 0.0100
- link Frame_FHC2: mass 0 -> 0.0100
- link Frame_FHC2_FOV: mass 0 -> 0.0100
- link Frame_FHC3: mass 0 -> 0.0100
- link Frame_FHC3_FOV: mass 0 -> 0.0100
- link Frame_FHC4: mass 0 -> 0.0100
- link Frame_FHC4_FOV: mass 0 -> 0.0100
- link Frame_FHCB: mass 0 -> 0.0100
- link Frame_GDRT: mass 0 -> 0.0100
- link Frame_HGAG: mass 0 -> 0.0100
- link Frame_HGAS: mass 0 -> 0.0100
- link Frame_HS: mass 0 -> 0.0100
- link Frame_ICU: mass 0 -> 0.0100
- link Frame_MAZ: mass 0 -> 0.0100
- link Frame_MCL: mass 0 -> 0.0100
- link Frame_MCR: mass 0 -> 0.0100
- link Frame_MEL: mass 0 -> 0.0100
- link Frame_MI: mass 0 -> 0.0100
- link Frame_MOXIE: mass 0 -> 0.0100
- link Frame_NCL: mass 0 -> 0.0100
- link Frame_NCL_FOV: mass 0 -> 0.0100
- link Frame_NCR: mass 0 -> 0.0100
- link Frame_NCR_FOV: mass 0 -> 0.0100
- link Frame_PIXL: mass 0 -> 0.0100
- link Frame_RA1: mass 0 -> 0.0100
- link Frame_RA2: mass 0 -> 0.0100
- link Frame_RA3: mass 0 -> 0.0100
- link Frame_RA4: mass 0 -> 0.0100
- link Frame_RA5: mass 0 -> 0.0100
- link Frame_RA6: mass 0 -> 0.0100
- link Frame_RA_BASE: mass 0 -> 0.0100
- link Frame_RDS: mass 0 -> 0.0100
- link Frame_RHC1: mass 0 -> 0.0100
- link Frame_RHC1_FOV: mass 0 -> 0.0100
- link Frame_RHC2: mass 0 -> 0.0100
- link Frame_RHC2_FOV: mass 0 -> 0.0100
- link Frame_RIMFAX: mass 0 -> 0.0100
- link Frame_RIMUA: mass 0 -> 0.0100
- link Frame_RIMUB: mass 0 -> 0.0100
- link Frame_RMECH: mass 0 -> 0.0100
- link Frame_RNAV: mass 0 -> 0.0100
- link Frame_ROCKER_L: mass 0 -> 0.0100
- link Frame_ROCKER_R: mass 0 -> 0.0100
- link Frame_SCI: mass 0 -> 0.0100
- link Frame_SCIR: mass 0 -> 0.0100
- link Frame_SCLIBS: mass 0 -> 0.0100
- link Frame_SCRMI: mass 0 -> 0.0100
- link Frame_SHERLOC: mass 0 -> 0.0100
- link Frame_STEER_LF: mass 0 -> 0.0100
- link Frame_STEER_LR: mass 0 -> 0.0100
- link Frame_STEER_RF: mass 0 -> 0.0100
- link Frame_STEER_RR: mass 0 -> 0.0100
- link Frame_TIRS: mass 0 -> 0.0100
- link Frame_TURRET: mass 0 -> 0.0100
- link Frame_WATSON: mass 0 -> 0.0100
- link Frame_WHEEL_LF: mass 0 -> 0.0100
- link Frame_WHEEL_LM: mass 0 -> 0.0100
- link Frame_WHEEL_LR: mass 0 -> 0.0100
- link Frame_WHEEL_RF: mass 0 -> 0.0100
- link Frame_WHEEL_RM: mass 0 -> 0.0100
- link Frame_WHEEL_RR: mass 0 -> 0.0100
- link Frame_WS1: mass 0 -> 0.0100
- link Frame_WS2: mass 0 -> 0.0100
- link ground: mass 0 -> 0.0100

Commit message: make robotic arm code to comments, but we can restore it very easilty and whenever we want

File: rover/m2020.urdf (robot description, URDF)
Before this commit: robot Perseverance, 115 links, 114 joints
Links:
- removed link Body_CorerFeed
- removed link Body_RA_Base
- removed link Body_RA_Link1
- removed link Body_RA_Link2
- removed link Body_RA_Link3
- removed link Body_RA_Link4
- removed link Body_RA_Link5
- removed link Body_SHERLOC_Cap
- removed link Body_StabilizerFar
- removed link Body_StabilizerNear
- removed link Body_Turret
- removed link Body_WATSON_Cap
- removed link Frame_CAL_PIXL
- removed link Frame_CAL_SHERLOC
- removed link Frame_DOCKING_POST
- removed link Frame_DRILL
- removed link Frame_FCS
- removed link Frame_GDRT
- removed link Frame_PIXL
- removed link Frame_RA1
- removed link Frame_RA2
- removed link Frame_RA3
- removed link Frame_RA4
- removed link Frame_RA5
- removed link Frame_RA6
- removed link Frame_RA_BASE
- removed link Frame_SHERLOC
- removed link Frame_TURRET
- removed link Frame_WATSON
Joints:
- removed joint DRILL_FEED
- removed joint JOINT1_ENC
- removed joint JOINT2_ENC
- removed joint JOINT3_ENC
- removed joint JOINT4_ENC
- removed joint JOINT5_ENC
- removed joint JointRobotArmBase
- removed joint JointTurret
- removed joint Joint_for_Frame_CAL_PIXL
- removed joint Joint_for_Frame_CAL_SHERLOC
- removed joint Joint_for_Frame_DOCKING_POST
- removed joint Joint_for_Frame_DRILL
- removed joint Joint_for_Frame_FCS
- removed joint Joint_for_Frame_GDRT
- removed joint Joint_for_Frame_PIXL
- removed joint Joint_for_Frame_RA1
- removed joint Joint_for_Frame_RA2
- removed joint Joint_for_Frame_RA3
- removed joint Joint_for_Frame_RA4
- removed joint Joint_for_Frame_RA5
- removed joint Joint_for_Frame_RA6
- removed joint Joint_for_Frame_RA_BASE
- removed joint Joint_for_Frame_SHERLOC
- removed joint Joint_for_Frame_TURRET
- removed joint Joint_for_Frame_WATSON
- removed joint SHERLOC_CAP_ENC
- removed joint STABILIZER_LOWER
- removed joint STABILIZER_UPPER
- removed joint WATSON_CAP_ENC

Commit message: URDF Rewrite for ROS coordinate system

File: rover/m2020.urdf (robot description, URDF)
Before this commit: robot Perseverance, 86 links, 85 joints
Joints:
- joint CENTER_DIFFERENTIAL: axis 0 0 1 -> 0 0 -1.0; origin xyz=-0.05198 0 -1.13338 rpy=0 -0 0 -> xyz=-0.05198 0 1.13338 rpy=0 0 0
- joint HGA_AZ: axis 0 0 1 -> 0 0 -1.0; origin xyz=-0.36998 -0.475 -1.13288 rpy=0 -0 0.436332 -> xyz=-0.36998 0.475 1.13288 rpy=0 0 -0.43633200000000005
- joint HGA_EL: axis 1 0 0 -> 1.0 0 0; origin xyz=0 0 -0.248 rpy=0.785398 -0 0 -> xyz=0 0 0.248 rpy=0.785398 0 0
- joint JointRoot: origin xyz=0 0 0 rpy=0 -0 0 -> xyz=0 0 0 rpy=0 0 0
- joint Joint_MHS_DebrisShield: origin xyz=0.09002 0 -1.13338 rpy=0 -0 0 -> xyz=0.09002 0 1.13338 rpy=0 0 0
- joint Joint_for_Frame_ANT: origin xyz=0.2084 0 0 rpy=2.35619 -0 0 -> xyz=0.2084 0 0 rpy=2.35619 0 0
- joint Joint_for_Frame_ATS1: origin xyz=0.846027 0.597543 -1.44188 rpy=1.5708 -0 2.44323 -> xyz=0.846027 -0.597543 1.44188 rpy=1.5707999999999998 0 -2.44323
- joint Joint_for_Frame_ATS2: origin xyz=0.749647 0.576177 -1.49028 rpy=-1.5708 -0 1.13391 -> xyz=0.749647 -0.576177 1.49028 rpy=-1.5708 0 -1.13391
- joint Joint_for_Frame_ATS3: origin xyz=0.816326 0.50341 -1.44188 rpy=1.5708 -0 0.348992 -> xyz=0.816326 -0.50341 1.44188 rpy=1.5707999999999998 0 -0.34899199999999997
- joint Joint_for_Frame_ATS4: origin xyz=0.896872 -0.63405 -0.879074 rpy=-1.5708 -0 -1.5708 -> xyz=0.896872 0.63405 0.879074 rpy=-1.5707999999999998 5.551115123125783e-17 1.5707999999999998
- joint Joint_for_Frame_ATS5: origin xyz=0.896872 0.63405 -0.830674 rpy=1.5708 -0 1.5708 -> xyz=0.896872 -0.63405 0.830674 rpy=1.5707999999999998 5.551115123125783e-17 -1.5707999999999998
- joint Joint_for_Frame_BOGIE_L: origin xyz=0 0 0 rpy=-1.5708 -0 0 -> xyz=0 0 0 rpy=-1.5707999999999998 0 0
- joint Joint_for_Frame_BOGIE_R: origin xyz=0 0 0 rpy=-1.5708 -0 0 -> xyz=0 0 0 rpy=-1.5707999999999998 0 0
- joint Joint_for_Frame_CAL_MC1: origin xyz=-0.28518 0.414008 -1.30252 rpy=3.14159 -0 0 -> xyz=-0.28518 -0.414008 1.30252 rpy=3.14159 0 0
- joint Joint_for_Frame_CAL_MC2: origin xyz=-0.23089 0.436008 -1.26302 rpy=3.14159 -0 0 -> xyz=-0.23089 -0.436008 1.26302 rpy=3.14159 0 0
- joint Joint_for_Frame_CAL_SC: origin xyz=-0.73817 0.5365 -1.29482 rpy=2.26898 -0 1.5708 -> xyz=-0.73817 -0.5365 1.29482 rpy=2.2689799999999996 0 -1.5707999999999998
- joint Joint_for_Frame_DIFF: origin xyz=0 0 0 rpy=0 -0 0 -> xyz=0 0 0 rpy=0 0 0
- joint Joint_for_Frame_FHC1: origin xyz=1.03958 0.226094 -0.760608 rpy=-0.174841 1.117 -0.000247676 -> xyz=1.03958 -0.226094 0.760608 rpy=-0.1748409999999999 -1.1169999999999995 0.00024767599999999404
- joint Joint_for_Frame_FHC1_FOV: origin xyz=1.09534 0.237039 -0.733411 rpy=-0.174841 1.117 -0.000247676 -> xyz=1.09534 -0.237039 0.733411 rpy=-0.1748409999999999 -1.1169999999999995 0.00024767599999999404
- joint Joint_for_Frame_FHC2: origin xyz=1.05159 -0.002264 -0.754746 rpy=0.174841 1.117 0.000247676 -> xyz=1.05159 0.002264 0.754746 rpy=0.1748409999999999 -1.1169999999999995 -0.00024767599999999404
- joint Joint_for_Frame_FHC2_FOV: origin xyz=1.10736 -0.0132091 -0.727549 rpy=0.174841 1.117 0.000247676 -> xyz=1.10736 0.0132091 0.727549 rpy=0.1748409999999999 -1.1169999999999995 -0.00024767599999999404
- joint Joint_for_Frame_FHC3: origin xyz=1.05159 0.150264 -0.754746 rpy=-0.174841 1.117 -0.000247676 -> xyz=1.05159 -0.150264 0.754746 rpy=-0.1748409999999999 -1.1169999999999995 0.00024767599999999404
- joint Joint_for_Frame_FHC3_FOV: origin xyz=1.10736 0.161209 -0.727549 rpy=-0.174841 1.117 -0.000247676 -> xyz=1.10736 -0.161209 0.727549 rpy=-0.1748409999999999 -1.1169999999999995 0.00024767599999999404
- joint Joint_for_Frame_FHC4: origin xyz=1.03958 -0.078094 -0.760608 rpy=0.174841 1.117 0.000247676 -> xyz=1.03958 0.078094 0.760608 rpy=0.1748409999999999 -1.1169999999999995 -0.00024767599999999404
- joint Joint_for_Frame_FHC4_FOV: origin xyz=1.09534 -0.0890391 -0.733411 rpy=0.174841 1.117 0.000247676 -> xyz=1.09534 0.0890391 0.733411 rpy=0.1748409999999999 -1.1169999999999995 -0.00024767599999999404
- joint Joint_for_Frame_FHCB: origin xyz=0.95652 0.074 -0.76858 rpy=0 -0 0 -> xyz=0.95652 -0.074 0.76858 rpy=0 0 0
- joint Joint_for_Frame_HGAG: origin xyz=0 0 0 rpy=3.14159 -0 0 -> xyz=0 0 0 rpy=3.14159 0 0
- joint Joint_for_Frame_HGAS: origin xyz=-0.36998 -0.475 -1.13288 rpy=0 -0 0.436316 -> xyz=-0.36998 0.475 1.13288 rpy=0 0 -0.43631600000000004
- joint Joint_for_Frame_HS: origin xyz=0.743443 0.576337 -1.50598 rpy=-0.463643 1.57079 0.463643 -> xyz=0.743443 -0.576337 1.50598 rpy=-0.46364300003282255 -1.5707900000454242 -0.46364300000927955
- joint Joint_for_Frame_ICU: origin xyz=0.179008 -0.209 -1.04738 rpy=3.14159 -0 0 -> xyz=0.179008 0.209 1.04738 rpy=3.14159 0 0
- joint Joint_for_Frame_MAZ: origin xyz=0 0 0 rpy=0 -0 0 -> xyz=0 0 0 rpy=0 0 0
- joint Joint_for_Frame_MCL: origin xyz=-0.085135 -0.126634 -0.065127 rpy=0 -0 0.0219954 -> xyz=-0.085135 0.126634 0.065127 rpy=0 0 -0.0219954
- joint Joint_for_Frame_MCR: origin xyz=-0.085134 0.121506 -0.065128 rpy=0 -0 -0.0220028 -> xyz=-0.085134 -0.121506 0.065128 rpy=0 0 0.0220028
- joint Joint_for_Frame_MEL: origin xyz=0 0 0 rpy=-1.5708 -0 0 -> xyz=0 0 0 rpy=-1.5707999999999998 0 0
- joint Joint_for_Frame_MI: origin xyz=0.804037 0.559028 -1.13288 rpy=0 -0 0 -> xyz=0.804037 -0.559028 1.13288 rpy=0 0 0
- joint Joint_for_Frame_MOXIE: origin xyz=-0.193552 -0.508 -1.04738 rpy=0 -0 0 -> xyz=-0.193552 0.508 1.04738 rpy=0 0 0
- joint Joint_for_Frame_NCL: origin xyz=0.080595 -0.214392 -0.057109 rpy=1.57079 1.57079 1.57079 -> xyz=0.080595 0.214392 0.057109 rpy=1.5707899999855608 -1.5707899999576844 -1.5707899999855608
- joint Joint_for_Frame_NCL_FOV: origin xyz=0.143595 -0.214392 -0.057109 rpy=1.57079 1.57079 1.57079 -> xyz=0.143595 0.214392 0.057109 rpy=1.5707899999855608 -1.5707899999576844 -1.5707899999855608
- joint Joint_for_Frame_NCR: origin xyz=0.080595 0.209607 -0.057111 rpy=1.57079 1.57079 1.57079 -> xyz=0.080595 -0.209607 0.057111 rpy=1.5707899999855608 -1.5707899999576844 -1.5707899999855608
- joint Joint_for_Frame_NCR_FOV: origin xyz=0.143595 0.209607 -0.057111 rpy=1.57079 1.57079 1.57079 -> xyz=0.143595 -0.209607 0.057111 rpy=1.5707899999855608 -1.5707899999576844 -1.5707899999855608
- joint Joint_for_Frame_RDS: origin xyz=0.138992 -0.298597 -1.17948 rpy=3.14159 -2.64698e-23 -0.157044 -> xyz=0.138992 0.298597 1.17948 rpy=3.14159 2.6469779601696886e-23 0.15704400000000002
- joint Joint_for_Frame_RHC1: origin xyz=-1.00766 -0.467 -0.77468 rpy=-2.99453e-22 0.785336 3.14159 -> xyz=-1.00766 0.467 0.77468 rpy=-2.9945275602387965e-22 -0.785336 -3.14159
- joint Joint_for_Frame_RHC1_FOV: origin xyz=-1.0522 -0.467 -0.73013 rpy=-2.99453e-22 0.785336 3.14159 -> xyz=-1.0522 0.467 0.73013 rpy=-2.9945275602387965e-22 -0.785336 -3.14159
- joint Joint_for_Frame_RHC2: origin xyz=-1.00766 0.467 -0.77468 rpy=-2.99453e-22 0.785336 3.14159 -> xyz=-1.00766 -0.467 0.77468 rpy=-2.9945275602387965e-22 -0.785336 -3.14159
- joint Joint_for_Frame_RHC2_FOV: origin xyz=-1.0522 0.467 -0.73013 rpy=-2.99453e-22 0.785336 3.14159 -> xyz=-1.0522 -0.467 0.73013 rpy=-2.9945275602387965e-22 -0.785336 -3.14159
- joint Joint_for_Frame_RIMFAX: origin xyz=-0.79478 0 -0.71724 rpy=-0.686834 -5.55112e-17 1.5708 -> xyz=-0.79478 0 0.71724 rpy=-0.686834 5.551115123125783e-17 -1.5707999999999998
- joint Joint_for_Frame_RIMUA: origin xyz=0.310906 -0.441586 -1.04738 rpy=0 0 -1.5708 -> xyz=0.310906 0.441586 1.04738 rpy=0 0 1.5707999999999998
- joint Joint_for_Frame_RIMUB: origin xyz=0.403906 -0.441586 -1.04738 rpy=0 0 -1.5708 -> xyz=0.403906 0.441586 1.04738 rpy=0 0 1.5707999999999998
- joint Joint_for_Frame_RMECH: origin xyz=0.09002 0 -1.13338 rpy=0 -0 0 -> xyz=0.09002 0 1.13338 rpy=0 0 0
- joint Joint_for_Frame_RNAV: origin xyz=0 0 0 rpy=0 -0 0 -> xyz=0 0 0 rpy=0 0 0
- joint Joint_for_Frame_ROCKER_L: origin xyz=0 0 0 rpy=-1.5708 -0 0 -> xyz=0 0 0 rpy=-1.5707999999999998 0 0
- joint Joint_for_Frame_ROCKER_R: origin xyz=0 0 0 rpy=-1.5708 -0 0 -> xyz=0 0 0 rpy=-1.5707999999999998 0 0
- joint Joint_for_Frame_SCI: origin xyz=-0.071379 -0.112 -0.114609 rpy=3.14159 -0 0 -> xyz=-0.071379 0.112 0.114609 rpy=3.14159 0 0
- joint Joint_for_Frame_SCIR: origin xyz=-0.062479 -0.112 -0.213609 rpy=3.14159 -0 0 -> xyz=-0.062479 0.112 0.213609 rpy=3.14159 0 0
- joint Joint_for_Frame_SCLIBS: origin xyz=-0.062479 -0.112 -0.213609 rpy=3.14159 -0 0 -> xyz=-0.062479 0.112 0.213609 rpy=3.14159 0 0
- joint Joint_for_Frame_SCRMI: origin xyz=-0.062479 -0.112 -0.213609 rpy=3.14159 -0 0 -> xyz=-0.062479 0.112 0.213609 rpy=3.14159 0 0
- joint Joint_for_Frame_STEER_LF: origin xyz=0 0 0 rpy=0 -0 0 -> xyz=0 0 0 rpy=0 0 0
- joint Joint_for_Frame_STEER_LR: origin xyz=0 0 0 rpy=0 -0 0 -> xyz=0 0 0 rpy=0 0 0
- joint Joint_for_Frame_STEER_RF: origin xyz=0 0 0 rpy=0 -0 0 -> xyz=0 0 0 rpy=0 0 0
- joint Joint_for_Frame_STEER_RR: origin xyz=0 0 0 rpy=0 -0 0 -> xyz=0 0 0 rpy=0 0 0
- joint Joint_for_Frame_TIRS: origin xyz=0.802591 0.616374 -1.55388 rpy=0 -0 -1.53621 -> xyz=0.802591 -0.616374 1.55388 rpy=0 0 1.53621
- joint Joint_for_Frame_WHEEL_LF: origin xyz=0 0 0 rpy=0 -0 0 -> xyz=0 0 0 rpy=0 0 0
- joint Joint_for_Frame_WHEEL_LM: origin xyz=0 0 0 rpy=0 -0 0 -> xyz=0 0 0 rpy=0 0 0
- joint Joint_for_Frame_WHEEL_LR: origin xyz=0 0 0 rpy=0 -0 0 -> xyz=0 0 0 rpy=0 0 0
- joint Joint_for_Frame_WHEEL_RF: origin xyz=0 0 0 rpy=0 -0 0 -> xyz=0 0 0 rpy=0 0 0
- joint Joint_for_Frame_WHEEL_RM: origin xyz=0 0 0 rpy=0 -0 0 -> xyz=0 0 0 rpy=0 0 0
- joint Joint_for_Frame_WHEEL_RR: origin xyz=0 0 0 rpy=0 -0 0 -> xyz=0 0 0 rpy=0 0 0
- joint Joint_for_Frame_WS1: origin xyz=0.854257 0.597514 -1.59588 rpy=0 -0 0.104166 -> xyz=0.854257 -0.597514 1.59588 rpy=0 0 -0.10416599999999998
- joint Joint_for_Frame_WS2: origin xyz=0.801386 0.623898 -1.62438 rpy=0 -0 2.19924 -> xyz=0.801386 -0.623898 1.62438 rpy=0 0 -2.19924
- joint LEFT_BOGIE: axis 0 1 0 -> 0 -1.0 0; origin xyz=-0.754 -0.12 0.23 rpy=0 -0 0 -> xyz=-0.754 0.12 -0.23 rpy=0 0 0
- joint LEFT_DIFFERENTIAL: axis 0 1 0 -> 0 -1.0 0; origin xyz=0.30402 -0.79959 -0.89288 rpy=0 -0 0 -> xyz=0.30402 0.79959 0.89288 rpy=0 0 0
- joint LF_DRIVE: axis 0 -1 0 -> 0 1.0 0; origin xyz=0 0 0 rpy=0 -0 0 -> xyz=0 0 0 rpy=0 0 0
- joint LF_STEER: axis 0 0 1 -> 0 0 -1.0; origin xyz=0.881 -0.26291 0.63 rpy=0 -0 0 -> xyz=0.881 0.26291 -0.63 rpy=0 0 0
- joint LM_DRIVE: axis 0 -1 0 -> 0 1.0 0; origin xyz=0.44998 -0.26491 0.4 rpy=0 -0 0 -> xyz=0.44998 0.26491 -0.4 rpy=0 0 0
- joint LR_DRIVE: axis 0 -1 0 -> 0 1.0 0; origin xyz=0 0 0 rpy=0 -0 0 -> xyz=0 0 0 rpy=0 0 0
- joint LR_STEER: axis 0 0 1 -> 0 0 -1.0; origin xyz=-0.625 -0.14291 0.4 rpy=0 -0 0 -> xyz=-0.625 0.14291 -0.4 rpy=0 0 0
- joint RF_DRIVE: axis 0 -1 0 -> 0 1.0 0; origin xyz=0 0 0 rpy=0 -0 0 -> xyz=0 0 0 rpy=0 0 0
- joint RF_STEER: axis 0 0 1 -> 0 0 -1.0; origin xyz=0.881 0.26291 0.63 rpy=0 -0 0 -> xyz=0.881 -0.26291 -0.63 rpy=0 0 0
- joint RIGHT_BOGIE: axis 0 1 0 -> 0 -1.0 0; origin xyz=-0.754 0.12 0.23 rpy=0 -0 0 -> xyz=-0.754 -0.12 -0.23 rpy=0 0 0
- joint RIGHT_DIFFERENTIAL: axis 0 1 0 -> 0 -1.0 0; origin xyz=0.30402 0.79959 -0.89288 rpy=0 -0 0 -> xyz=0.30402 -0.79959 0.89288 rpy=0 0 0
- joint RM_DRIVE: axis 0 -1 0 -> 0 1.0 0; origin xyz=0.44998 0.26491 0.4 rpy=0 -0 0 -> xyz=0.44998 -0.26491 -0.4 rpy=0 0 0
- joint RR_DRIVE: axis 0 -1 0 -> 0 1.0 0; origin xyz=0 0 0 rpy=0 -0 0 -> xyz=0 0 0 rpy=0 0 0
- joint RR_STEER: axis 0 0 1 -> 0 0 -1.0; origin xyz=-0.625 0.14291 0.4 rpy=0 -0 0 -> xyz=-0.625 -0.14291 -0.4 rpy=0 0 0
- joint RSM_AZ_ENC: axis 0 0 1 -> 0 0 -1.0; origin xyz=0.804037 0.559028 -1.91927 rpy=0 -0 3.12414 -> xyz=0.804037 -0.559028 1.91927 rpy=0 0 -3.12414
- joint RSM_EL_ENC: axis 0 1 0 -> 0 -1.0 0; origin xyz=0 0 0 rpy=3.14159 -1.55334 3.14159 -> xyz=0 0 0 rpy=3.14159 1.5533399999999986 -3.14159
